Commit message: [update] new galbot

File: env/data/assets/galbot_one_simplified/galbot_one_10_DoF.urdf (robot description, URDF)
Before this commit: robot galbot_one, 51 links, 50 joints
Links:
- added link left_gripper_acronym_link
- link left_arm_camera_flange_link: geometry 
Joints:
- added joint acronym_joint: type fixed, parent left_gripper_base_link, child left_gripper_acronym_link, origin xyz=0 0 0.070 rpy=0 0 0, axis 0 0 0

File: env/data/assets/galbot_one_simplified/galbot_one_7_DoF.urdf (robot description, URDF)
Before this commit: robot galbot_one, 51 links, 50 joints
Links:
- added link left_gripper_acronym_link
Joints:
- added joint acronym_joint: type fixed, parent left_gripper_base_link, child left_gripper_acronym_link, origin xyz=0 0 0.070 rpy=0 0 0, axis 0 0 0

Commit message: [update] camera position

File: env/data/assets/galbot_one_simplified/galbot_one_10_DoF.urdf (robot description, URDF)
Before this commit: robot galbot_one, 52 links, 51 joints
Links:
- added link front_head_camera_color_optical_frame
- added link left_arm_camera_color_optical_frame
Joints:
- added joint front_camera_joint_calibration: type fixed, parent right_arm_base_link, child front_head_camera_color_optical_frame, origin xyz=0.07244318503551352 0.2536318547766252 -0.17073446195851838 rpy=2.8390350174780554 -1.5371566014113576 -0.13187440313966659, axis 0 0 0
- added joint left_arm_camera_joint_calibration: type fixed, parent left_arm_end_effector_mount_link, child left_arm_camera_color_optical_frame, origin xyz=-0.03723097546064943 0.057109830265918086 0.024428711356245303 rpy=0.26058160947492603 0.0012649375988844636 -2.042211434373371, axis 0 0 0

Commit message: [fix] camera rotation

File: env/data/assets/galbot_one_simplified/galbot_one_10_DoF.urdf (robot description, URDF)
Before this commit: robot galbot_one, 54 links, 53 joints
Links:
- link head_base_link: geometry 
- link head_link1: geometry 
- link head_link2: geometry 
